Commit message: feat(gazebo): 添加传感器模型和rviz配置文件到gazebo仿真功能包中

File: gazebo_simulation/robots/sentry2026.urdf.xacro (robot description, xacro)
@@ -179,4 +179,71 @@
     <dynamics damping="0.05" friction="0.0"/>
   </joint>
+  <!-- MID-360 mount copied from simple_livox.urdf.xacro. -->
+  <link name="mid360_link">
+    <visual>
+      <geometry>
+        <mesh filename="package://gazebo_simulation/models/mid360/meshes/mid360.dae"/>
+      </geometry>
+      <material name="light_gray"/>
+    </visual>
+    <collision name="mid360_collision">
+      <geometry><box size="0.08 0.12 0.08"/></geometry>
+    </collision>
+    <inertial>
+      <mass value="1.0"/>
+      <inertia ixx="0.1" ixy="0" ixz="0"
+               iyy="0.1" iyz="0" izz="0.1"/>
+    </inertial>
+  </link>
+  <joint name="mid360_mount_joint" type="fixed">
+    <parent link="gimbal_yaw_big_link"/>
+    <child link="mid360_link"/>
+    <origin xyz="0.0668 -0.1623 0.1195" rpy="0 0 0"/>
+  </joint>
+  <!-- Sensor parameters are taken from models/mid360/model.sdf. -->
+  <gazebo reference="mid360_link">
+    <gravity>false</gravity>
+    <sensor name="mid360_lidar" type="gpu_lidar">
+      <ignition_frame_id>mid360_link</ignition_frame_id>
+      <pose>0 0 0.03 0 0 0</pose>
+      <topic>/model/sentry/mid360/scan</topic>
+      <always_on>true</always_on>
+      <visualize>true</visualize>
+      <update_rate>10.0</update_rate>
+      <ray>
+        <scan>
+          <horizontal>
+            <samples>1500</samples>
+            <resolution>1</resolution>
+            <min_angle>0</min_angle>
+            <max_angle>6.2831852</max_angle>
+          </horizontal>
+          <vertical>
+            <samples>32</samples>
+            <resolution>1</resolution>
+            <min_angle>-0.12217304764</min_angle>
+            <max_angle>0.90757121104</max_angle>
+          </vertical>
+        </scan>
+        <range>
+          <min>0.15</min>
+          <max>15.0</max>
+          <resolution>0.01</resolution>
+        </range>
+      </ray>
+      <noise>
+        <type>gaussian</type>
+        <mean>0.0</mean>
+        <stddev>0.01</stddev>
+      </noise>
+    </sensor>
+    <sensor name="mid360_imu" type="imu">
+      <ignition_frame_id>mid360_link</ignition_frame_id>
+      <topic>/model/sentry/mid360/imu</topic>
+      <always_on>true</always_on>
+      <visualize>true</visualize>
+      <update_rate>200</update_rate>
+    </sensor>
+  </gazebo>
   <gazebo reference="chassis_link">
     <gravity>true</gravity>
@@ -286,4 +353,8 @@
         <tf_topic>/model/sentry/pose</tf_topic>
       </plugin>
+      <plugin filename="gz-sim-joint-state-publisher-system"
+              name="gz::sim::systems::JointStatePublisher">
+        <topic>/world/default/model/sentry/joint_state</topic>
+      </plugin>
     </gazebo>
   </xacro:if>
